Commit message: Updated reflection axis wheels

File: ros_dude_description/urdf/dude.urdf.xacro (robot description, xacro)
@@ -192,8 +192,8 @@
   <!-- Asus Xtion Pro Live -->
   <!-- Wheels -->
-  <xacro:banebots_wheel position="left">
+  <xacro:banebots_wheel position="left" reflect="1">
     <origin xyz="${wheel_offset_x} ${-wheel_offset_y} ${wheel_offset_z}" rpy="${M_PI/2} 0 0" />
   </xacro:banebots_wheel>
-  <xacro:banebots_wheel position="right">
+  <xacro:banebots_wheel position="right" reflect="-1">
     <origin xyz="${wheel_offset_x} ${wheel_offset_y} ${wheel_offset_z}" rpy="${-M_PI/2} 0 0" />
   </xacro:banebots_wheel>

File: ros_dude_description/urdf/wheel.urdf.xacro (robot description, xacro)
@@ -1,5 +1,5 @@
 <?xml version="1.0"?>
 <robot xmlns:xacro="http://ros.org/wiki/xacro" name="dude_wheel">
-  <xacro:macro name="banebots_wheel" params="position *joint_pose">
+  <xacro:macro name="banebots_wheel" params="position reflect *joint_pose">
     <link name="${position}_wheel_link">
       <visual>
@@ -11,7 +11,7 @@
       </visual>
       <collision>
-        <origin xyz="0 0 0" rpy="${M_PI/2} 0 0" />
+        <origin xyz="0 0 0" rpy="0 0 0" />
         <geometry>
-          <mesh filename="package://ros_dude_description/meshes/wheel/wheel_link.STL" />
+          <cylinder length="${wheel_leght}" radius="${wheel_radius}"/>
         </geometry>
       </collision>
@@ -20,9 +20,6 @@
         <mass value="0.0372140206710188" />
         <inertia
-          ixx="1.12116949143941E-05"
-          ixy="-4.09082423865234E-22"
-          ixz="1.90582413132218E-21"
-          iyy="2.18923205916391E-05"
-          iyz="-1.28651410234429E-21"
+          ixx="1.12116949143941E-05" ixy="0" ixz="0"
+          iyy="2.18923205916391E-05" iyz="0"
           izz="1.12116949143941E-05" />
       </inertial>
@@ -34,4 +31,5 @@
       <kd value="1.0" />
       <fdir1 value="1 0 0"/>
+      <maxContacts>1</maxContacts>
       <material>Gazebo/Blue</material>
     </gazebo>
@@ -42,5 +40,5 @@
       <joint_properties damping="0.0" friction="0.0"/>
       <xacro:insert_block name="joint_pose"/>
-      <axis xyz="0 0 1"/>
+      <axis xyz="0 0 ${reflect}"/>
     </joint>
   </xacro:macro>

Commit message: Added Transmission and confuration for ros control

File: ros_dude_description/urdf/dude.urdf.xacro (robot description, xacro)
@@ -191,8 +191,8 @@
   <!-- Asus Xtion Pro Live -->
   <!-- Wheels -->
-  <xacro:banebots_wheel position="left" reflect="1">
+  <xacro:banebots_wheel position="left" reflect="-1">
     <origin xyz="${wheel_offset_x} ${-wheel_offset_y} ${wheel_offset_z}" rpy="${M_PI/2} 0 0" />
   </xacro:banebots_wheel>
-  <xacro:banebots_wheel position="right" reflect="-1">
+  <xacro:banebots_wheel position="right" reflect="1">
     <origin xyz="${wheel_offset_x} ${wheel_offset_y} ${wheel_offset_z}" rpy="${-M_PI/2} 0 0" />
   </xacro:banebots_wheel>

File: ros_dude_description/urdf/wheel.urdf.xacro (robot description, xacro)
@@ -42,4 +42,14 @@
       <axis xyz="0 0 ${reflect}"/>
     </joint>
+		<transmission name="${position}_trans" type="SimpleTransmission">
+			<type>transmission_interface/SimpleTransmission</type>
+			<actuator name="${position}_motor">
+				<hardwareInterface>EffortJointInterface</hardwareInterface>
+				<mechanicalReduction>1</mechanicalReduction>
+			</actuator>
+			<joint name="${position}">
+				<hardwareInterface>EffortJointInterface</hardwareInterface>
+			</joint>
+		</transmission>
   </xacro:macro>
 </robot>
