Commit message: Fixed information about driver control

File: ros_dude_description/urdf/wheel.urdf.xacro (robot description, xacro)
@@ -37,5 +37,5 @@
       <parent link="base_link"/>
       <child link="${position}_wheel_link"/>
-      <limit effort="100" velocity="100"/>
+      <limit effort="100" velocity="12"/>
       <joint_properties damping="0.0" friction="0.0"/>
       <xacro:insert_block name="joint_pose"/>
