Commit message: Added gazebo color

File: ros_dude_description/urdf/asus_xtion_pro.urdf.xacro (robot description, xacro)
@@ -73,4 +73,10 @@
     <axis xyz="0 0 0" />
   </joint>
+  <gazebo reference="xtion_sensor">
+    <material>Gazebo/Black</material>
+  </gazebo>
+  <gazebo reference="xtion_camera">
+    <material>Gazebo/Black</material>
+  </gazebo>
   </xacro:macro>
 </robot>

File: ros_dude_description/urdf/description.xacro (robot description, xacro)
@@ -24,18 +24,3 @@
   <xacro:include filename="$(find ros_dude_description)/urdf/dude.urdf.xacro" />
   <xacro:dude_robot />
-	<!--<gazebo>
-		<plugin name="differential_drive_controller" filename="libgazebo_ros_diff_drive.so">
-		  <alwaysOn>true</alwaysOn>
-		  <updateRate>10.0</updateRate>
-		  <leftJoint>Right</leftJoint>
-		  <rightJoint>Left</rightJoint>
-		  <wheelSeparation>0.5380</wheelSeparation>
-		  <wheelDiameter>0.2410</wheelDiameter>
-		  <torque>20</torque>
-		  <commandTopic>cmd_vel</commandTopic>
-		  <odometryTopic>odom</odometryTopic>
-		  <odometryFrame>odom</odometryFrame>
-		  <robotBaseFrame>base_link</robotBaseFrame>
-		</plugin>
-	</gazebo>-->
 </robot>

File: ros_dude_description/urdf/dude.urdf.xacro (robot description, xacro)
@@ -195,5 +195,5 @@
     <origin xyz="${wheel_offset_x} ${-wheel_offset_y} ${wheel_offset_z}" rpy="${M_PI/2} 0 0" />
   </xacro:banebots_wheel>
-  <xacro:banebots_wheel position="Right">
+  <xacro:banebots_wheel position="right">
     <origin xyz="${wheel_offset_x} ${wheel_offset_y} ${wheel_offset_z}" rpy="${-M_PI/2} 0 0" />
   </xacro:banebots_wheel>

File: ros_dude_description/urdf/omniwheel.urdf.xacro (robot description, xacro)
@@ -35,4 +35,7 @@
     <axis xyz="0 -1 0" />
   </joint>
+  <gazebo reference="omniwheel">
+    <material>Gazebo/DarkGrey</material>
+  </gazebo>
   <link name="wheel1_omniwheel_Link">
     <inertial>
@@ -67,4 +70,7 @@
     <axis xyz="-1 0 0" />
   </joint>
+  <gazebo reference="wheel1_omniwheel">
+    <material>Gazebo/Black</material>
+  </gazebo>
   <link name="wheel2_omniwheel_Link">
     <inertial>
@@ -99,4 +105,7 @@
     <axis xyz="-1 0 0" />
   </joint>
+  <gazebo reference="wheel2_omniwheel">
+    <material>Gazebo/Black</material>
+  </gazebo>
   <link name="wheel3_omniwheel_Link">
     <inertial>
@@ -131,4 +140,7 @@
     <axis xyz="-1 0 0" />
   </joint>
+  <gazebo reference="wheel3_omniwheel">
+    <material>Gazebo/Black</material>
+  </gazebo>
   <link name="wheel4_omniwheel_Link">
     <inertial>
@@ -163,4 +175,7 @@
     <axis xyz="-1 0 0" />
   </joint>
+  <gazebo reference="wheel4_omniwheel">
+    <material>Gazebo/Black</material>
+  </gazebo>
   <link name="wheel5_omniwheel_Link">
     <inertial>
@@ -195,4 +210,7 @@
     <axis xyz="-1 0 0" />
   </joint>
+  <gazebo reference="wheel5_omniwheel">
+    <material>Gazebo/Black</material>
+  </gazebo>
   <link name="wheel6_omniwheel_Link">
     <inertial>
@@ -227,4 +245,7 @@
     <axis xyz="-1 0 0" />
   </joint>
+  <gazebo reference="wheel6_omniwheel">
+    <material>Gazebo/Black</material>
+  </gazebo>
   <link name="wheel7_omniwheel_Link">
     <inertial>
@@ -259,4 +280,7 @@
     <axis xyz="-1 0 0" />
   </joint>
+  <gazebo reference="wheel7_omniwheel">
+    <material>Gazebo/Black</material>
+  </gazebo>
   <link name="wheel8_omniwheel_Link">
     <inertial>
@@ -291,4 +315,7 @@
     <axis xyz="-1 0 0" />
   </joint>
+  <gazebo reference="wheel8_omniwheel">
+    <material>Gazebo/Black</material>
+  </gazebo>
   </xacro:macro>
 </robot>

File: ros_dude_description/urdf/wheel.urdf.xacro (robot description, xacro)
@@ -4,18 +4,18 @@
     <link name="${position}_wheel_link">
       <visual>
-				<origin xyz="0 0 0" rpy="${M_PI/2} 0 0" />
-      <geometry>
-        <mesh filename="package://ros_dude_description/meshes/wheel/wheel_link.STL" />
-      </geometry>
-        <material name="Blue" />
+        <origin xyz="0 0 0" rpy="${M_PI/2} 0 0" />
+          <geometry>
+            <mesh filename="package://ros_dude_description/meshes/wheel/wheel_link.STL" />
+          </geometry>
+          <material name="Blue" />
       </visual>
       <collision>
-				<origin xyz="0 0 0" rpy="${M_PI/2} 0 0" />
-      <geometry>
-        <mesh filename="package://ros_dude_description/meshes/wheel/wheel_link.STL" />
-      </geometry>
+        <origin xyz="0 0 0" rpy="${M_PI/2} 0 0" />
+        <geometry>
+          <mesh filename="package://ros_dude_description/meshes/wheel/wheel_link.STL" />
+        </geometry>
       </collision>
       <inertial>
-        <origin xyz="-6.93889390390723E-18 6.54344632364662E-05 6.93889390390723E-18" rpy="0 0 0" />
+        <origin xyz="-6.93889390390723E-18 6.54344632364662E-05 6.93889390390723E-18" rpy="${M_PI/2} 0 0" />
         <mass value="0.0372140206710188" />
         <inertia
@@ -28,11 +28,12 @@
       </inertial>
     </link>
-		<gazebo reference="${position}_wheel_link">
-			<mu1 value="1.0"/>
-			<mu2 value="1.0"/>
-			<kp value="10000000.0" />
-			<kd value="1.0" />
-			<fdir1 value="1 0 0"/>
-		</gazebo>
+    <gazebo reference="${position}_wheel_link">
+      <mu1 value="1.0"/>
+      <mu2 value="1.0"/>
+      <kp value="10000000.0" />
+      <kd value="1.0" />
+      <fdir1 value="1 0 0"/>
+      <material>Gazebo/Blue</material>
+    </gazebo>
     <joint name="${position}" type="continuous">
       <parent link="base_link"/>

Commit message: Updated mesh robot

File: ros_dude_description/urdf/asus_xtion_pro.urdf.xacro (robot description, xacro)
@@ -1,40 +1,31 @@
 <?xml version="1.0"?>
 <robot name="sensor_asus_xtion_pro" xmlns:xacro="http://ros.org/wiki/xacro">
-  <!-- Xacro properties -->
-  <xacro:property name="M_SCALE" value="0.001"/>
-  <xacro:property name="asus_xtion_pro_depth_rel_rgb_py" value="0.0270" />
-  <xacro:property name="asus_xtion_pro_cam_rel_rgb_py"   value="-0.0220" />
-  <xacro:property name="path" value="package://ros_dude_description/meshes/xtion" />
   <!-- Parameterised in part by the values in turtlebot_properties.urdf.xacro -->
-  <xacro:macro name="sensor_asus_xtion_pro" params="parent">
+  <xacro:macro name="sensor_asus_xtion_pro" params="parent type *joint_pose">
   <link name="xtion_sensor_Link">
     <inertial>
-      <origin xyz="-5.24598794596834E-05 -0.00118587892274831 -8.67757641544151E-07" rpy="0 0 0" />
-      <mass value="0.0157220883907246" />
+      <origin xyz="0.00025226 0 0.0028141" rpy="0 0 0" />
+      <mass value="0.015722" />
       <inertia
-        ixx="1.04171049584748E-05"
-        ixy="1.28442051710763E-10"
-        ixz="1.18967372459655E-11"
-        iyy="1.19900865482375E-05"
-        iyz="-6.38594842692275E-13"
-        izz="1.91603460288645E-06" />
+        ixx="1.0417E-05" ixy="-1.1897E-11" ixz="-1.2844E-10"
+        iyy="1.916E-06" iyz="-6.3859E-13"
+        izz="1.199E-05" />
     </inertial>
     <visual>
       <origin xyz="0 0 0" rpy="0 0 0" />
       <geometry>
-        <mesh filename="${path}/xtion_sensor_Link.STL" />
+        <mesh filename="${path_meshes}/xtion/xtion_sensor_Link.STL" />
       </geometry>
       <material name="Black" />
     </visual>
     <collision>
-      <origin xyz="0 0 0" rpy="0 0 0" />
+      <origin xyz="0 0 0.02" rpy="0 0 0" />
       <geometry>
-        <mesh filename="${path}/xtion_sensor_Link.STL" />
+        <box size="0.015 0.015 0.04"/>
       </geometry>
     </collision>
   </link>
   <joint name="xtion_sensor" type="fixed">
-    <!--<origin xyz="0.00451431691853688 0 0.116837599999998" rpy="1.5707963267949 0 0" />-->
-    <origin xyz="${cam_px} ${cam_py} ${cam_pz}" rpy="${cam_or} ${cam_op} ${cam_oy}"/>
+    <xacro:insert_block name="joint_pose"/>
     <parent link="${parent}" />
     <child link="xtion_sensor_Link" />
@@ -43,33 +34,38 @@
   <link name="xtion_camera_Link">
     <inertial>
-      <origin xyz="0.00279241240109677 0.0211137711711282 -0.00708713336677233" rpy="0 0 0" />
-      <mass value="0.150306955527936" />
+      <origin xyz="-0.00077984 -0.00028713 0.021283" rpy="0 0 0" />
+      <mass value="0.15031" />
       <inertia
-        ixx="0.00039934046078429"
-        ixy="-6.26137198523733E-07"
-        ixz="5.31643806851641E-07"
-        iyy="0.000406006690758908"
-        iyz="-5.93032579916887E-08"
-        izz="2.36182089627434E-05" />
+        ixx="0.00039928" ixy="-5.3487E-07" ixz="-1.3724E-08"
+        iyy="2.3618E-05" iyz="-8.6762E-09"
+        izz="0.00040606" />
     </inertial>
     <visual>
       <origin xyz="0 0 0" rpy="0 0 0" />
       <geometry>
-        <mesh filename="${path}/xtion_camera_Link.STL" />
+        <mesh filename="${path_meshes}/xtion/xtion_camera_Link.STL" />
       </geometry>
       <material name="Black" />
     </visual>
     <collision>
-      <origin xyz="0 0 0" rpy="0 0 0" />
+      <origin xyz="0 0 0.021" rpy="0 0 0" />
       <geometry>
-        <mesh filename="${path}/xtion_camera_Link.STL" />
+        <box size="0.035 0.18 0.022"/>
       </geometry>
     </collision>
   </link>
-  <joint name="xtion_camera" type="fixed">
-    <origin xyz="-6.43169185368941E-05 0.0087500000000001 0.00679918490215687" rpy="0 0 0" />
+    <gazebo reference="xtion_camera_Link">
+      <mu1 value="1.0"/>
+      <mu2 value="1.0"/>
+      <kp value="10000000.0" />
+      <kd value="1.0" />
+      <fdir1 value="1 0 0"/>
+    </gazebo>
+  <joint name="xtion_camera" type="${type}">
+    <origin xyz="0.00026411 0 0.01275" rpy="0 0 0" />
     <parent link="xtion_sensor_Link" />
     <child link="xtion_camera_Link" />
-    <axis xyz="0 0 0" />
+    <limit effort="1000.0" lower="-0.68" upper="0.68" velocity="0.5"/>
+    <axis xyz="0 -1 0" />
   </joint>
   <gazebo reference="xtion_sensor">

File: ros_dude_description/urdf/dude.urdf.xacro (robot description, xacro)
@@ -3,9 +3,11 @@
   <!-- Included URDF/XACRO Files -->
   <xacro:include filename="$(find ros_dude_description)/urdf/materials.urdf" />
+  <xacro:include filename="$(find ros_dude_description)/urdf/motor.urdf.xacro" />
+  <xacro:include filename="$(find ros_dude_description)/urdf/omniwheel.urdf.xacro" />
   <xacro:include filename="$(find ros_dude_description)/urdf/wheel.urdf.xacro" />
-  <xacro:include filename="$(find ros_dude_description)/urdf/omniwheel.urdf.xacro" />
   <xacro:include filename="$(find ros_dude_description)/urdf/asus_xtion_pro.urdf.xacro"/>
   <!-- Included URDF/XACRO Files -->
   <!-- Global properties -->
+  <property name="path_meshes" value="package://ros_dude_description/meshes"/>
   <property name="M_PI" value="3.14159"/>
   <!-- Global properties -->
@@ -18,8 +20,9 @@
   <!-- Wheels params -->
   <!-- Asus Xtion params -->
-  <property name="cam_px" value="0.004" />
+  <property name="camera_axis" value="fixed"/>
+  <property name="cam_px" value="-0.005" />
   <property name="cam_py" value="0.0" />
-  <property name="cam_pz" value="0.117" />
-  <property name="cam_or" value="${M_PI/2}" />
+  <property name="cam_pz" value="0.113" />
+  <property name="cam_or" value="0" />
   <property name="cam_op" value="0" />
   <property name="cam_oy" value="0" />
@@ -27,100 +30,48 @@
   <!-- base_link -->
   <link name="base_link">
-    <visual>
-      <origin xyz="0 0 0" rpy="0 0 0" />
-      <geometry>
-        <mesh filename="package://ros_dude_description/meshes/body/base_link.STL" />
+    <inertial>
+      <origin xyz="-0.08572 0 0.034445" rpy="0 0 0" />
+      <mass value="0.43258" />
+      <inertia
+        ixx="0.0013149" ixy="0" ixz="0.00013884"
+        iyy="0.0021698" iyz="0"
+        izz="0.0028089" />
+    </inertial>
+    <visual>
+      <origin xyz="0 0 0" rpy="0 0 0" />
+      <geometry>
+        <mesh filename="${path_meshes}/body/base_link.STL" />
       </geometry>
       <material name="Yellow" />
     </visual>
     <collision>
-      <origin xyz="0 0 0" rpy="0 0 0" />
-      <geometry>
-        <mesh filename="package://ros_dude_description/meshes/body/base_link.STL" />
+      <origin xyz="0.0 0.0 0.07" rpy="0 0 0" />
+      <geometry>
+        <box size="0.08 0.14 0.11"/>
       </geometry>
     </collision>
-    <inertial>
-      <origin xyz="0.0857197083472489 4.15321029299353E-06 0.0344447185380985" rpy="0 0 0" />
-      <mass value="0.432580623668397" />
-      <inertia
-        ixx="0.00131485031864629"
-        ixy="-1.43314122310053E-07"
-        ixz="-0.00013883510641213"
-        iyy="0.0021697759965098"
-        iyz="5.7298696577375E-08"
-        izz="0.0028089452261539" />
-    </inertial>
+    <collision>
+      <origin xyz="-0.13 0.0 0.07" rpy="0 0 0" />
+      <geometry>
+        <box size="0.18 0.19 0.11"/>
+      </geometry>
+    </collision>
   </link>
   <!-- base_link -->
   <!-- Body chassis -->
-  <link name="column_body_Link">
-    <visual>
-      <origin xyz="0 0 0" rpy="0 0 0" />
-      <geometry>
-        <mesh filename="package://ros_dude_description/meshes/body/column_body_Link.STL" />
-      </geometry>
-      <material name="Black" />
-    </visual>
-    <collision>
-      <origin xyz="0 0 0" rpy="0 0 0" />
-      <geometry>
-        <mesh filename="package://ros_dude_description/meshes/body/column_body_Link.STL" />
-      </geometry>
-    </collision>
-    <inertial>
-      <origin xyz="0.0907213301786849 -0.00088772159450999 0.0311173420281291" rpy="0 0 0" />
-      <mass value="0.186878289960642" />
-      <inertia
-        ixx="0.000527558823944031"
-        ixy="9.5073271246689E-06"
-        ixz="-2.48756139563941E-05"
-        iyy="0.00132787178905797"
-        iyz="-4.31040060828821E-06"
-        izz="0.00174484068650444" />
-    </inertial>
-  </link>
-  <joint name="column_body" type="fixed">
-    <origin xyz="-0.03105 0 0.0138375999999985" rpy="6.12303176911189E-17 0 0" />
-    <parent link="base_link" />
-    <child link="column_body_Link" />
-    <axis xyz="0 0 0" />
-  </joint>
-  <link name="electronics_Link">
-    <visual>
-      <origin xyz="0 0 0" rpy="0 0 0" />
-      <geometry>
-        <mesh filename="package://ros_dude_description/meshes/body/electronics_Link.STL" />
-      </geometry>
-      <material name="Green" />
-    </visual>
-    <collision>
-      <origin xyz="0 0 0" rpy="0 0 0" />
-      <geometry>
-        <mesh filename="package://ros_dude_description/meshes/body/electronics_Link.STL" />
-      </geometry>
-    </collision>
-    <inertial>
-      <origin xyz="0.138900427528209 -0.0024010475998454 0.0686403397577923" rpy="0 0 0" />
-      <mass value="0.0598796777354097" />
-      <inertia
-        ixx="7.76258699993621E-05"
-        ixy="1.65741409241155E-05"
-        ixz="6.34984589085961E-06"
-        iyy="0.000128840758819345"
-        iyz="1.77979090945961E-06"
-        izz="0.00020266312793241" />
-    </inertial>
-  </link>
-  <joint name="electronics" type="fixed">
-    <origin xyz="-0.03105 0 0.0138375999999985" rpy="6.12303176911189E-17 0 0" />
-    <parent link="base_link" />
-    <child link="electronics_Link" />
-    <axis xyz="0 0 0" />
-  </joint>
   <link name="wall_body_Link">
-    <visual>
-      <origin xyz="0 0 0" rpy="0 0 0" />
-      <geometry>
-        <mesh filename="package://ros_dude_description/meshes/body/wall_body_Link.STL" />
+    <inertial>
+      <origin xyz="-0.090836 0 0.084998" rpy="0 0 0" />
+      <mass value="0.20283" />
+      <inertia
+        ixx="0.0009070" ixy="0" ixz="0"
+        iyy="0.0012807" iyz="0"
+        izz="0.0017437" />
+    </inertial>
+    <visual>
+      <origin xyz="0 0 0" rpy="0 0 0" />
+      <geometry>
+        <mesh
+          filename="${path_meshes}/body/wall_body_Link.STL" />
       </geometry>
       <material name="">
@@ -128,65 +79,120 @@
       </material>
     </visual>
-    <collision>
-      <origin xyz="0 0 0" rpy="0 0 0" />
-      <geometry>
-        <mesh filename="package://ros_dude_description/meshes/body/wall_body_Link.STL" />
-      </geometry>
-    </collision>
-    <inertial>
-      <origin xyz="0.121885567097329 8.96585445430196E-05 0.071160775843539" rpy="0 0 0" />
-      <mass value="0.20282613968088" />
-      <inertia
-        ixx="0.000907087574558297"
-        ixy="-9.64733356695E-08"
-        ixz="1.39027570885642E-06"
-        iyy="0.00128070018487064"
-        iyz="1.21595625127852E-07"
-        izz="0.00174365625531033" />
-    </inertial>
   </link>
   <joint name="wall_body" type="fixed">
-    <origin xyz="-0.03105 0 0.0138375999999985" rpy="6.12303176911189E-17 0 0" />
+    <origin xyz="0 0 0" rpy="0 0 0" />
     <parent link="base_link" />
     <child link="wall_body_Link" />
     <axis xyz="0 0 0" />
   </joint>
+  <link name="column_body_Link">
+    <inertial>
+      <origin xyz="-0.10613 0.0015789 0.046254" rpy="0 0 0" />
+      <mass value="0.10507" />
+      <inertia
+        ixx="0.00033714" ixy="0" ixz="0"
+        iyy="0.00079716" iyz="0"
+        izz="0.0010369" />
+    </inertial>
+    <visual>
+      <origin xyz="0 0 0" rpy="0 0 0" />
+      <geometry>
+        <mesh filename="${path_meshes}/body/column_body_Link.STL" />
+      </geometry>
+      <material name="Black" />
+    </visual>
+  </link>
+  <joint name="column_body" type="fixed">
+    <origin xyz="0 0 0" rpy="0 0 0" />
+    <parent link="base_link" />
+    <child link="column_body_Link" />
+    <axis xyz="0 0 0" />
+  </joint>
   <link name="battery_Link">
-    <visual>
-      <origin xyz="0 0 0" rpy="0 0 0" />
-      <geometry>
-        <mesh filename="package://ros_dude_description/meshes/body/battery_Link.STL" />
-      </geometry>
-      <material name="Black" />
-    </visual>
-    <collision>
-      <origin xyz="0 0 0" rpy="0 0 0" />
-      <geometry>
-        <mesh filename="package://ros_dude_description/meshes/body/battery_Link.STL" />
-      </geometry>
-    </collision>
-    <inertial>
-      <origin xyz="0 -0.018 0" rpy="0 0 0" />
-      <mass value="0.24980980400259" />
-      <inertia
-        ixx="0.000444825252242251"
-        ixy="-1.06032793940047E-21"
-        ixz="-9.67661265350208E-21"
-        iyy="0.000468434653970205"
-        iyz="0"
-        izz="7.63561548404154E-05" />
-    </inertial>
+    <inertial>
+      <origin xyz="0 0 0.018" rpy="0 0 0" />
+      <mass value="0.24981" />
+      <inertia
+        ixx="0.00044483" ixy="1.2332E-20" ixz="1.0603E-21"
+        iyy="7.6356E-05" iyz="2.4007E-20"
+        izz="0.00046843" />
+    </inertial>
+    <visual>
+      <origin xyz="0 0 0" rpy="0 0 0" />
+      <geometry>
+        <mesh filename="${path_meshes}/body/battery_Link.STL" />
+      </geometry>
+      <material name="Blue" />
+    </visual>
   </link>
   <joint name="battery" type="fixed">
-    <origin xyz="0.08145 0 0.0558375999999985" rpy="1.5707963267949 0 0" />
+    <origin xyz="-0.08145 0 0.0198375999999985" rpy="0 0 0" />
     <parent link="base_link" />
     <child link="battery_Link" />
     <axis xyz="0 0 0" />
   </joint>
+  <link name="electronics_Link">
+    <inertial>
+      <origin xyz="-0.036996 0.030509 0.06534" rpy="0 0 0" />
+      <mass value="0.0041313" />
+      <inertia
+        ixx="5.2552E-07" ixy="4.4197E-12" ixz="3.55E-11"
+        iyy="5.2551E-07" iyz="7.1007E-11"
+        izz="1.0455E-06" />
+    </inertial>
+    <visual>
+      <origin xyz="0 0 0" rpy="0 0 0" />
+      <geometry>
+        <mesh filename="${path_meshes}/body/electronics_Link.STL" />
+      </geometry>
+      <material name="White" />
+    </visual>
+  </link>
+  <joint name="electronics" type="fixed">
+    <origin xyz="0.03105 0 0.0138375999999985" rpy="0 0 0" />
+    <parent link="base_link" />
+    <child link="electronics_Link" />
+    <axis xyz="0 0 0" />
+  </joint>
+  <link name="jetson_board_Link">
+    <inertial>
+      <origin xyz="-0.014974 0.000698 0.0046671" rpy="0 0 0" />
+      <mass value="0.054421" />
+      <inertia
+        ixx="7.5163E-05" ixy="4.1299E-06" ixz="-4.9228E-06"
+        iyy="8.1481E-05" iyz="-1.4961E-06"
+        izz="0.00015315" />
+    </inertial>
+    <visual>
+      <origin xyz="0 0 0" rpy="0 0 0" />
+      <geometry>
+        <mesh filename="${path_meshes}/body/jetson_board_Link.STL" />
+      </geometry>
+      <material name="Green" />
+    </visual>
+  </link>
+  <joint name="jetson_board" type="fixed">
+    <origin xyz="-0.131461588151754 0 0.064" rpy="0 0 0" />
+    <parent link="electronics_Link" />
+    <child link="jetson_board_Link" />
+    <axis xyz="0 0 0" />
+  </joint>
+  <!-- Motors -->
+  <xacro:motor position="left" parent="column_body_Link">
+    <origin xyz="0 0.087616 0.0365" rpy="0 0 0" />
+  </xacro:motor>
+  <xacro:motor position="right" parent="column_body_Link">
+    <origin xyz="0 -0.087616 0.0365" rpy="0 0 ${M_PI}" />
+  </xacro:motor>
+  <!-- Motors -->
   <!-- Omniwheel -->
-  <xacro:omniwheel parent="base_link"/>
+  <xacro:omniwheel parent="base_link">
+    <origin xyz="-0.20895 0 0.021838" rpy="0 0 ${M_PI}" />
+  </xacro:omniwheel>
   <!-- Omniwheel -->
   <!-- Asus Xtion Pro Live -->
-  <xacro:sensor_asus_xtion_pro parent="base_link"/>
+  <xacro:sensor_asus_xtion_pro parent="base_link" type="${camera_axis}">
+    <origin xyz="${cam_px} ${cam_py} ${cam_pz}"  rpy="${cam_or} ${cam_op} ${cam_oy}" />
+  </xacro:sensor_asus_xtion_pro>
   <!-- Asus Xtion Pro Live -->
   <!-- Wheels -->
