Commit message: Updated mesh robot

File: ros_dude_description/urdf/omniwheel.urdf.xacro (robot description, xacro)
@@ -1,321 +1,44 @@
 <?xml version="1.0"?>
-<robot xmlns:xacro="http://ros.org/wiki/xacro" name="dude_wheel">
-  <xacro:property name="path_omniwheel" value="package://ros_dude_description/meshes/omniwheel" />
-  <xacro:macro name="omniwheel" params="parent">
-  <link name="omniwheel_Link">
-    <inertial>
-      <origin xyz="-2.98078228766485E-12 -0.0159999999998262 1.04373801268487E-12" rpy="0 0 0" />
-      <mass value="0.0164743786019311" />
-      <inertia
-        ixx="2.5182162984259E-06"
-        ixy="-1.6301814784866E-16"
-        ixz="-2.08449514363363E-21"
-        iyy="2.61137234386137E-06"
-        iyz="5.75450229214032E-17"
-        izz="2.51596416456903E-06" />
-    </inertial>
-    <visual>
-      <origin xyz="0 0 0" rpy="0 0 0" />
-      <geometry>
-        <mesh filename="${path_omniwheel}/omniwheel_Link.STL" />
-      </geometry>
-      <material name="DarkGrey" />
-    </visual>
-    <collision>
-      <origin xyz="0 0 0" rpy="0 0 0" />
-      <geometry>
-        <mesh filename="${path_omniwheel}/omniwheel_Link.STL" />
-      </geometry>
-    </collision>
-  </link>
-  <joint name="omniwheel" type="continuous">
-    <origin xyz="0.20895 0.016 0.0218375999999985" rpy="0 0 0" />
-    <parent link="${parent}" />
-    <child link="omniwheel_Link" />
-    <axis xyz="0 -1 0" />
-  </joint>
-  <gazebo reference="omniwheel">
-    <material>Gazebo/DarkGrey</material>
-  </gazebo>
-  <link name="wheel1_omniwheel_Link">
-    <inertial>
-      <origin xyz="-0.0109250000000001 1.66533453693773E-16 1.73472347597681E-18" rpy="0 0 0" />
-      <mass value="0.00151452717448798" />
-      <inertia
-        ixx="2.51251046593801E-08"
-        ixy="-2.14239778651234E-22"
-        ixz="-6.91875383716808E-25"
-        iyy="3.99451464831259E-08"
-        iyz="2.80707627581717E-26"
-        izz="3.99451464831259E-08" />
-    </inertial>
-    <visual>
-      <origin xyz="0 0 0" rpy="0 0 0" />
-      <geometry>
-        <mesh filename="${path_omniwheel}/wheel1_omniwheel_Link.STL" />
-      </geometry>
-      <material name="Black" />
-    </visual>
-    <collision>
-      <origin xyz="0 0 0" rpy="0 0 0" />
-      <geometry>
-        <mesh filename="${path_omniwheel}/wheel1_omniwheel_Link.STL" />
-      </geometry>
-    </collision>
-  </link>
-  <joint name="wheel1_omniwheel" type="continuous">
-    <origin xyz="0.015604857543621 -0.008 0.00910825803258154" rpy="1.5707963267949 0.394916918533723 -9.26825791289139E-17" />
-    <parent link="omniwheel_Link" />
-    <child link="wheel1_omniwheel_Link" />
-    <axis xyz="-1 0 0" />
-  </joint>
-  <gazebo reference="wheel1_omniwheel">
-    <material>Gazebo/Black</material>
-  </gazebo>
-  <link name="wheel2_omniwheel_Link">
-    <inertial>
-      <origin xyz="0.0108739898732232 -1.94289029309402E-16 0" rpy="0 0 0" />
-      <mass value="0.00151452717448798" />
-      <inertia
-        ixx="2.51251046593798E-08"
-        ixy="2.36573655190166E-22"
-        ixz="1.81385736627921E-25"
-        iyy="3.99451464831245E-08"
-        iyz="3.52788837746716E-26"
-        izz="3.99451464831245E-08" />
-    </inertial>
-    <visual>
-      <origin xyz="0 0 0" rpy="0 0 0" />
-      <geometry>
-        <mesh filename="${path_omniwheel}/wheel2_omniwheel_Link.STL" />
-      </geometry>
-      <material name="Black" />
-    </visual>
-    <collision>
-      <origin xyz="0 0 0" rpy="0 0 0" />
-      <geometry>
-        <mesh filename="${path_omniwheel}/wheel2_omniwheel_Link.STL" />
-      </geometry>
-    </collision>
-  </link>
-  <joint name="wheel2_omniwheel" type="continuous">
-    <origin xyz="0.0174950161828645 -0.008 0.00451623206955716" rpy="1.5707963267949 1.17587940826117 3.14159265358979" />
-    <parent link="omniwheel_Link" />
-    <child link="wheel2_omniwheel_Link" />
-    <axis xyz="-1 0 0" />
-  </joint>
-  <gazebo reference="wheel2_omniwheel">
-    <material>Gazebo/Black</material>
-  </gazebo>
-  <link name="wheel3_omniwheel_Link">
-    <inertial>
-      <origin xyz="0.0108739898732232 -1.66533453693773E-16 0" rpy="0 0 0" />
-      <mass value="0.00151452717448798" />
-      <inertia
-        ixx="2.51251046593813E-08"
-        ixy="2.27474668452083E-22"
-        ixz="-1.46188663777651E-24"
-        iyy="3.9945146483125E-08"
-        iyz="-2.36488835798662E-26"
-        izz="3.9945146483125E-08" />
-    </inertial>
-    <visual>
-      <origin xyz="0 0 0" rpy="0 0 0" />
-      <geometry>
-        <mesh filename="${path_omniwheel}/wheel3_omniwheel_Link.STL" />
-      </geometry>
-      <material name="Black" />
-    </visual>
-    <collision>
-      <origin xyz="0 0 0" rpy="0 0 0" />
-      <geometry>
-        <mesh filename="${path_omniwheel}/wheel3_omniwheel_Link.STL" />
-      </geometry>
-    </collision>
-  </link>
-  <joint name="wheel3_omniwheel" type="continuous">
-    <origin xyz="0.00451623206955709 -0.008 -0.0174950161828646" rpy="1.5707963267949 -0.39491691853373 3.14159265358979" />
-    <parent link="omniwheel_Link" />
-    <child link="wheel3_omniwheel_Link" />
-    <axis xyz="-1 0 0" />
-  </joint>
-  <gazebo reference="wheel3_omniwheel">
-    <material>Gazebo/Black</material>
-  </gazebo>
-  <link name="wheel4_omniwheel_Link">
-    <inertial>
-      <origin xyz="0.0108739898732231 1.38777878078145E-16 0" rpy="0 0 0" />
-      <mass value="0.00151452717448798" />
-      <inertia
-        ixx="2.51251046593761E-08"
-        ixy="-2.01004888850386E-22"
-        ixz="-4.33511020203432E-25"
-        iyy="3.99451464831227E-08"
-        iyz="-1.26291076632911E-27"
-        izz="3.99451464831227E-08" />
-    </inertial>
-    <visual>
-      <origin xyz="0 0 0" rpy="0 0 0" />
-      <geometry>
-        <mesh filename="${path_omniwheel}/wheel4_omniwheel_Link.STL" />
-      </geometry>
-      <material name="Black" />
-    </visual>
-    <collision>
-      <origin xyz="0 0 0" rpy="0 0 0" />
-      <geometry>
-        <mesh filename="${path_omniwheel}/wheel4_omniwheel_Link.STL" />
-      </geometry>
-    </collision>
-  </link>
-  <joint name="wheel4_omniwheel" type="continuous">
-    <origin xyz="-0.0174950161828646 -0.008 -0.00451623206955703" rpy="1.5707963267949 -1.17587940826116 -3.37828843903879E-17" />
-    <parent link="omniwheel_Link" />
-    <child link="wheel4_omniwheel_Link" />
-    <axis xyz="-1 0 0" />
-  </joint>
-  <gazebo reference="wheel4_omniwheel">
-    <material>Gazebo/Black</material>
-  </gazebo>
-  <link name="wheel5_omniwheel_Link">
-    <inertial>
-      <origin xyz="0.0108739898732234 8.32667268468867E-17 0" rpy="0 0 0" />
-      <mass value="0.00151452717448798" />
-      <inertia
-        ixx="2.51251046593813E-08"
-        ixy="1.24077091882954E-22"
-        ixz="-5.4144158476139E-25"
-        iyy="3.99451464831257E-08"
-        iyz="1.14426806846713E-25"
-        izz="3.99451464831257E-08" />
-    </inertial>
-    <visual>
-      <origin xyz="0 0 0" rpy="0 0 0" />
-      <geometry>
-        <mesh filename="${path_omniwheel}/wheel5_omniwheel_Link.STL" />
-      </geometry>
-      <material name="Black" />
-    </visual>
-    <collision>
-      <origin xyz="0 0 0" rpy="0 0 0" />
-      <geometry>
-        <mesh filename="${path_omniwheel}/wheel5_omniwheel_Link.STL" />
-      </geometry>
-    </collision>
-  </link>
-  <joint name="wheel5_omniwheel" type="continuous">
-    <origin xyz="0.0091773862580764 -0.024 0.0155643029016678" rpy="1.5707963267949 1.18031508193121 -1.34779352725226E-16" />
-    <parent link="omniwheel_Link" />
-    <child link="wheel5_omniwheel_Link" />
-    <axis xyz="-1 0 0" />
-  </joint>
-  <gazebo reference="wheel5_omniwheel">
-    <material>Gazebo/Black</material>
-  </gazebo>
-  <link name="wheel6_omniwheel_Link">
-    <inertial>
-      <origin xyz="0.0108739898732234 -2.77555756156289E-17 -1.73472347597681E-18" rpy="0 0 0" />
-      <mass value="0.00151452717448798" />
-      <inertia
-        ixx="2.51251046593799E-08"
-        ixy="-1.24077091882954E-22"
-        ixz="-1.68544304494927E-24"
-        iyy="3.99451464831246E-08"
-        iyz="-7.27783536444543E-26"
-        izz="3.99451464831246E-08" />
-    </inertial>
-    <visual>
-      <origin xyz="0 0 0" rpy="0 0 0" />
-      <geometry>
-        <mesh filename="${path_omniwheel}/wheel6_omniwheel_Link.STL" />
-      </geometry>
-      <material name="Black" />
-    </visual>
-    <collision>
-      <origin xyz="0 0 0" rpy="0 0 0" />
-      <geometry>
-        <mesh filename="${path_omniwheel}/wheel6_omniwheel_Link.STL" />
-      </geometry>
-    </collision>
-  </link>
-  <joint name="wheel6_omniwheel" type="continuous">
-    <origin xyz="0.0155643029016678 -0.024 -0.00917738625807647" rpy="1.5707963267949 0.390481244863686 3.14159265358979" />
-    <parent link="omniwheel_Link" />
-    <child link="wheel6_omniwheel_Link" />
-    <axis xyz="-1 0 0" />
-  </joint>
-  <gazebo reference="wheel6_omniwheel">
-    <material>Gazebo/Black</material>
-  </gazebo>
-  <link name="wheel7_omniwheel_Link">
-    <inertial>
-      <origin xyz="0.0108739898732234 5.55111512312578E-17 0" rpy="0 0 0" />
-      <mass value="0.00151452717448798" />
-      <inertia
-        ixx="2.51251046593786E-08"
-        ixy="-1.63781761285499E-22"
-        ixz="-1.46758763574446E-24"
-        iyy="3.99451464831247E-08"
-        iyz="-1.12577022334281E-25"
-        izz="3.99451464831247E-08" />
-    </inertial>
-    <visual>
-      <origin xyz="0 0 0" rpy="0 0 0" />
-      <geometry>
-        <mesh filename="${path_omniwheel}/wheel7_omniwheel_Link.STL" />
-      </geometry>
-      <material name="Black" />
-    </visual>
-    <collision>
-      <origin xyz="0 0 0" rpy="0 0 0" />
-      <geometry>
-        <mesh filename="${path_omniwheel}/wheel7_omniwheel_Link.STL" />
-      </geometry>
-    </collision>
-  </link>
-  <joint name="wheel7_omniwheel" type="continuous">
-    <origin xyz="-0.00917738625807635 -0.024 -0.0155643029016679" rpy="1.5707963267949 -1.1803150819312 3.14159265358979" />
-    <parent link="omniwheel_Link" />
-    <child link="wheel7_omniwheel_Link" />
-    <axis xyz="-1 0 0" />
-  </joint>
-  <gazebo reference="wheel7_omniwheel">
-    <material>Gazebo/Black</material>
-  </gazebo>
-  <link name="wheel8_omniwheel_Link">
-    <inertial>
-      <origin xyz="-0.010925 1.38777878078145E-16 1.73472347597681E-18" rpy="0 0 0" />
-      <mass value="0.00151452717448798" />
-      <inertia
-        ixx="2.5125104659377E-08"
-        ixy="-5.9557004103818E-23"
-        ixz="-7.39970794498117E-25"
-        iyy="3.99451464831238E-08"
-        iyz="-2.19396873665366E-26"
-        izz="3.99451464831238E-08" />
-    </inertial>
-    <visual>
-      <origin xyz="0 0 0" rpy="0 0 0" />
-      <geometry>
-        <mesh filename="${path_omniwheel}/wheel8_omniwheel_Link.STL" />
-      </geometry>
-      <material name="Black" />
-    </visual>
-    <collision>
-      <origin xyz="0 0 0" rpy="0 0 0" />
-      <geometry>
-        <mesh filename="${path_omniwheel}/wheel8_omniwheel_Link.STL" />
-      </geometry>
-    </collision>
-  </link>
-  <joint name="wheel8_omniwheel" type="continuous">
-    <origin xyz="0.00459378956890963 -0.024 0.0174748116081796" rpy="1.5707963267949 -0.390481244863705 -7.53548068257853E-17" />
-    <parent link="omniwheel_Link" />
-    <child link="wheel8_omniwheel_Link" />
-    <axis xyz="-1 0 0" />
-  </joint>
-  <gazebo reference="wheel8_omniwheel">
-    <material>Gazebo/Black</material>
-  </gazebo>
+<robot xmlns:xacro="http://ros.org/wiki/xacro" name="omniwheel">
+  <xacro:macro name="omniwheel" params="parent *joint_pose">
+    <link name="omniwheel_Link">
+      <inertial>
+        <origin xyz="0 0 0" rpy="0 0 0" />
+        <mass value="0.028591" />
+        <inertia
+          ixx="4.812E-06" ixy="-1.630E-16" ixz="3.9705E-22"
+          iyy="5.447E-06" iyz="5.7548E-17"
+          izz="4.8098E-06" />
+      </inertial>
+      <visual>
+        <origin xyz="0 0 0" rpy="0 0 0" />
+        <geometry>
+          <mesh filename="${path_meshes}/omniwheel/omniwheel_Link.STL" />
+        </geometry>
+        <material name="DarkGrey" />
+      </visual>
+      <collision>
+        <origin xyz="0 0 0" rpy="0 0 0" />
+        <geometry>
+          <sphere radius="0.021"/>
+        </geometry>
+      </collision>
+    </link>
+    <gazebo reference="omniwheel_link">
+      <mu1 value="1.0"/>
+      <mu2 value="1.0"/>
+      <kp value="10000000.0" />
+      <kd value="1.0" />
+      <fdir1 value="1 0 0"/>
+      <maxContacts>1</maxContacts>
+      <material>Gazebo/Black</material>
+    </gazebo>
+    <joint name="omniwheel" type="continuous">
+      <xacro:insert_block name="joint_pose"/>
+      <parent link="${parent}" />
+      <child link="omniwheel_Link" />
+      <axis xyz="0 -1 0" />
+      <mimic joint="left" multiplier="1" offset="0"/>
+    </joint>
   </xacro:macro>
 </robot>

File: ros_dude_description/urdf/wheel.urdf.xacro (robot description, xacro)
@@ -6,5 +6,5 @@
         <origin xyz="0 0 0" rpy="${M_PI/2} 0 0" />
           <geometry>
-            <mesh filename="package://ros_dude_description/meshes/wheel/wheel_link.STL" />
+            <mesh filename="${path_meshes}/wheel/wheel_link.STL" />
           </geometry>
           <material name="Blue" />
@@ -17,5 +17,5 @@
       </collision>
       <inertial>
-        <origin xyz="-6.93889390390723E-18 6.54344632364662E-05 6.93889390390723E-18" rpy="${M_PI/2} 0 0" />
+        <origin xyz="0 0 0" rpy="${M_PI/2} 0 0" />
         <mass value="0.0372140206710188" />
         <inertia
@@ -42,14 +42,14 @@
       <axis xyz="0 0 ${reflect}"/>
     </joint>
-		<transmission name="${position}_trans" type="SimpleTransmission">
-			<type>transmission_interface/SimpleTransmission</type>
-			<actuator name="${position}_motor">
-				<hardwareInterface>EffortJointInterface</hardwareInterface>
-				<mechanicalReduction>1</mechanicalReduction>
-			</actuator>
-			<joint name="${position}">
-				<hardwareInterface>EffortJointInterface</hardwareInterface>
-			</joint>
-		</transmission>
+    <transmission name="${position}_trans" type="SimpleTransmission">
+      <type>transmission_interface/SimpleTransmission</type>
+      <actuator name="${position}_motor">
+        <hardwareInterface>EffortJointInterface</hardwareInterface>
+        <mechanicalReduction>1</mechanicalReduction>
+      </actuator>
+      <joint name="${position}">
+        <hardwareInterface>EffortJointInterface</hardwareInterface>
+      </joint>
+    </transmission>
   </xacro:macro>
 </robot>

Commit message: Added a new node for navigation. Added a new control in according with https://github.com/officinerobotiche/ros_serial_bridge/pull/20 and https://github.com/officinerobotiche/uNAV.X/pull/44 . Updated name xtion mesh

File: ros_dude_description/urdf/asus_xtion_pro.urdf.xacro (robot description, xacro)
@@ -1,7 +1,10 @@
 <?xml version="1.0"?>
 <robot name="sensor_asus_xtion_pro" xmlns:xacro="http://ros.org/wiki/xacro">
+  <!-- Xacro properties -->
+  <xacro:property name="asus_xtion_pro_depth_rel_rgb_py" value="0.0270" />
+  <xacro:property name="asus_xtion_pro_cam_rel_rgb_py"   value="-0.0220" />
   <!-- Parameterised in part by the values in turtlebot_properties.urdf.xacro -->
   <xacro:macro name="sensor_asus_xtion_pro" params="parent type *joint_pose">
-  <link name="xtion_sensor_Link">
+  <link name="xtion_sensor_link">
     <inertial>
       <origin xyz="0.00025226 0 0.0028141" rpy="0 0 0" />
@@ -15,5 +18,5 @@
       <origin xyz="0 0 0" rpy="0 0 0" />
       <geometry>
-        <mesh filename="${path_meshes}/xtion/xtion_sensor_Link.STL" />
+        <mesh filename="${path_meshes}/xtion/xtion_sensor_link.STL" />
       </geometry>
       <material name="Black" />
@@ -29,8 +32,8 @@
     <xacro:insert_block name="joint_pose"/>
     <parent link="${parent}" />
-    <child link="xtion_sensor_Link" />
+    <child link="xtion_sensor_link" />
     <axis xyz="0 0 0" />
   </joint>
-  <link name="xtion_camera_Link">
+  <link name="camera_link">
     <inertial>
       <origin xyz="-0.00077984 -0.00028713 0.021283" rpy="0 0 0" />
@@ -44,5 +47,5 @@
       <origin xyz="0 0 0" rpy="0 0 0" />
       <geometry>
-        <mesh filename="${path_meshes}/xtion/xtion_camera_Link.STL" />
+        <mesh filename="${path_meshes}/xtion/xtion_camera_link.STL" />
       </geometry>
       <material name="Black" />
@@ -55,5 +58,5 @@
     </collision>
   </link>
-    <gazebo reference="xtion_camera_Link">
+    <gazebo reference="camera_link">
       <mu1 value="1.0"/>
       <mu2 value="1.0"/>
@@ -64,13 +67,73 @@
   <joint name="xtion_camera" type="${type}">
     <origin xyz="0.00026411 0 0.01275" rpy="0 0 0" />
-    <parent link="xtion_sensor_Link" />
-    <child link="xtion_camera_Link" />
+    <parent link="xtion_sensor_link" />
+    <child link="camera_link" />
     <limit effort="1000.0" lower="-0.68" upper="0.68" velocity="0.5"/>
     <axis xyz="0 -1 0" />
   </joint>
+  <joint name="camera_rgb_joint" type="fixed">
+    <origin xyz="0 0.018 0.022" rpy="0 0 0" />
+    <parent link="camera_link"/>
+    <child link="camera_rgb_frame" />
+  </joint>
+  <link name="camera_rgb_frame"/>
+  <joint name="camera_rgb_optical_joint" type="fixed">
+    <origin xyz="0 0 0" rpy="${-M_PI/2} 0 ${-M_PI/2}" />
+    <parent link="camera_rgb_frame" />
+    <child link="camera_rgb_optical_frame" />
+  </joint>
+  <link name="camera_rgb_optical_frame"/>
+  <joint name="camera_depth_joint" type="fixed">
+    <origin xyz="0 ${asus_xtion_pro_depth_rel_rgb_py} 0" rpy="0 0 0" />
+    <parent link="camera_rgb_frame" />
+    <child link="camera_depth_frame" />
+  </joint>
+  <link name="camera_depth_frame"/>
+  <joint name="camera_depth_optical_joint" type="fixed">
+    <origin xyz="0 0 0" rpy="${-M_PI/2} 0 ${-M_PI/2}" />
+    <parent link="camera_depth_frame" />
+    <child link="camera_depth_optical_frame" />
+  </joint>
+  <link name="camera_depth_optical_frame"/>
+  <gazebo reference="camera_rgb_frame">
+    <sensor type="depth" name="camera">
+      <always_on>true</always_on>
+      <update_rate>20.0</update_rate>
+      <camera>
+        <horizontal_fov>${58.0*M_PI/180.0}</horizontal_fov>
+        <image>
+          <format>R8G8B8</format>
+          <width>640</width>
+          <height>480</height>
+        </image>
+        <clip>
+          <near>0.08</near>
+          <far>3.0</far>
+        </clip>
+      </camera>
+      <plugin name="camera_controller" filename="libgazebo_ros_openni_kinect.so">
+        <cameraName>camera</cameraName>
+        <alwaysOn>true</alwaysOn>
+        <updateRate>10</updateRate>
+        <imageTopicName>rgb/image_raw</imageTopicName>
+        <depthImageTopicName>depth/image_raw</depthImageTopicName>
+        <pointCloudTopicName>depth/points</pointCloudTopicName>
+        <cameraInfoTopicName>rgb/camera_info</cameraInfoTopicName>
+        <depthImageCameraInfoTopicName>depth/camera_info</depthImageCameraInfoTopicName>
+        <frameName>camera_rgb_optical_frame</frameName>
+        <baseline>0.1</baseline>
+        <distortion_k1>0.0</distortion_k1>
+        <distortion_k2>0.0</distortion_k2>
+        <distortion_k3>0.0</distortion_k3>
+        <distortion_t1>0.0</distortion_t1>
+        <distortion_t2>0.0</distortion_t2>
+        <pointCloudCutoff>0.4</pointCloudCutoff>
+      </plugin>
+    </sensor>
+  </gazebo>
   <gazebo reference="xtion_sensor">
     <material>Gazebo/Black</material>
   </gazebo>
-  <gazebo reference="xtion_camera">
+  <gazebo reference="camera">
     <material>Gazebo/Black</material>
   </gazebo>

File: ros_dude_description/urdf/dude.urdf.xacro (robot description, xacro)
@@ -197,8 +197,8 @@
   <!-- Asus Xtion Pro Live -->
   <!-- Wheels -->
-  <xacro:banebots_wheel position="left" reflect="-1">
+  <xacro:banebots_wheel position="Left" reflect="-1">
     <origin xyz="${wheel_offset_x} ${-wheel_offset_y} ${wheel_offset_z}" rpy="${M_PI/2} 0 0" />
   </xacro:banebots_wheel>
-  <xacro:banebots_wheel position="right" reflect="1">
+  <xacro:banebots_wheel position="Right" reflect="1">
     <origin xyz="${wheel_offset_x} ${wheel_offset_y} ${wheel_offset_z}" rpy="${-M_PI/2} 0 0" />
   </xacro:banebots_wheel>

File: ros_dude_description/urdf/omniwheel.urdf.xacro (robot description, xacro)
@@ -39,5 +39,5 @@
       <child link="omniwheel_Link" />
       <axis xyz="0 -1 0" />
-      <mimic joint="left" multiplier="1" offset="0"/>
+      <mimic joint="Left" multiplier="1" offset="0"/>
     </joint>
   </xacro:macro>
