Commit message: Updated xtion for laser scan

File: dude_description/urdf/asus_xtion_pro.urdf.xacro (robot description, xacro)
@@ -96,44 +96,4 @@
   </joint>
   <link name="rgbd_camera_depth_optical_frame"/>
-  <gazebo reference="rgbd_camera_rgb_frame">
-    <sensor type="depth" name="rgbd_camera">
-      <always_on>true</always_on>
-      <update_rate>20.0</update_rate>
-      <camera>
-        <horizontal_fov>${58.0*M_PI/180.0}</horizontal_fov>
-        <image>
-          <format>R8G8B8</format>
-          <width>640</width>
-          <height>480</height>
-        </image>
-        <clip>
-          <near>0.08</near>
-          <far>3.0</far>
-        </clip>
-      </camera>
-      <plugin name="camera_controller" filename="libgazebo_ros_openni_kinect.so">
-        <cameraName>rgbd_camera</cameraName>
-        <alwaysOn>true</alwaysOn>
-        <updateRate>10</updateRate>
-        <imageTopicName>rgb/image_raw</imageTopicName>
-        <depthImageTopicName>depth/image_raw</depthImageTopicName>
-        <pointCloudTopicName>depth/points</pointCloudTopicName>
-        <cameraInfoTopicName>rgb/camera_info</cameraInfoTopicName>
-        <depthImageCameraInfoTopicName>depth/camera_info</depthImageCameraInfoTopicName>
-        <frameName>rgbd_camera_rgb_optical_frame</frameName>
-        <baseline>0.1</baseline>
-        <distortion_k1>0.0</distortion_k1>
-        <distortion_k2>0.0</distortion_k2>
-        <distortion_k3>0.0</distortion_k3>
-        <distortion_t1>0.0</distortion_t1>
-        <distortion_t2>0.0</distortion_t2>
-        <pointCloudCutoff>0.4</pointCloudCutoff>
-      </plugin>
-    </sensor>
-    <material>Gazebo/Black</material>
-  </gazebo>
-  <gazebo reference="xtion_sensor">
-    <material>Gazebo/Black</material>
-  </gazebo>
   </xacro:macro>
 </robot>

File: dude_description/urdf/dude.urdf.xacro (robot description, xacro)
@@ -28,4 +28,5 @@
   <property name="cam_oy" value="0" />
   <!-- Asus Xtion params -->
+  <xacro:macro name="dude_robot">
   <!-- base_link -->
   <link name="base_link">
@@ -204,3 +205,4 @@
   </xacro:banebots_wheel>
   <!-- Wheels -->
+  </xacro:macro>
 </robot>
