Commit message: Moved launch file for unav and fixed torque for motor

File: dude_description/urdf/wheel.urdf.xacro (robot description, xacro)
@@ -37,5 +37,5 @@
       <parent link="base_link"/>
       <child link="${position}_wheel_link"/>
-      <limit effort="100" velocity="12"/>
+      <limit effort="12" velocity="12"/>
       <joint_properties damping="0.0" friction="0.0"/>
       <xacro:insert_block name="joint_pose"/>

Commit message: Added launch for exploration

File: dude_description/urdf/wheel.urdf.xacro (robot description, xacro)
@@ -37,5 +37,5 @@
       <parent link="base_link"/>
       <child link="${position}_wheel_link"/>
-      <limit effort="12" velocity="12"/>
+      <limit effort="12" velocity="25"/>
       <joint_properties damping="0.0" friction="0.0"/>
       <xacro:insert_block name="joint_pose"/>
