Commit message: Added first release of imu

File: dude_description/urdf/dude.urdf.xacro (robot description, xacro)
@@ -7,4 +7,5 @@
   <xacro:include filename="$(find dude_description)/urdf/wheel.urdf.xacro" />
   <xacro:include filename="$(find dude_description)/urdf/asus_xtion_pro.urdf.xacro"/>
+  <xacro:include filename="$(find dude_description)/urdf/imu.urdf.xacro"/>
   <!-- Included URDF/XACRO Files -->
   <!-- Global properties -->
@@ -179,4 +180,9 @@
     <axis xyz="0 0 0" />
   </joint>
+  <!-- IMU -->
+  <xacro:imu name="imu" parent="base_link">
+    <origin xyz="-0.06 0 0.11" rpy="0 0 0" />
+  </xacro:imu>
+  <!-- IMU -->
   <!-- Motors -->
   <xacro:motor position="left" parent="column_body_Link">

Commit message: Added dae file

File: dude_description/urdf/dude.urdf.xacro (robot description, xacro)
@@ -43,5 +43,5 @@
       <origin xyz="0 0 0" rpy="0 0 0" />
       <geometry>
-        <mesh filename="${path_meshes}/body/base_link.STL" />
+        <mesh filename="${path_meshes}/body/base_link.dae" />
       </geometry>
       <material name="Yellow" />

Commit message: Added IMU

File: dude_description/urdf/dude.urdf.xacro (robot description, xacro)
@@ -33,15 +33,15 @@
   <link name="base_link">
     <inertial>
-      <origin xyz="-0.08572 0 0.034445" rpy="0 0 0" />
-      <mass value="0.43258" />
-      <inertia
-        ixx="0.0013149" ixy="0" ixz="0.00013884"
-        iyy="0.0021698" iyz="0"
-        izz="0.0028089" />
-    </inertial>
-    <visual>
-      <origin xyz="0 0 0" rpy="0 0 0" />
-      <geometry>
-        <mesh filename="${path_meshes}/body/base_link.dae" />
+      <origin xyz="-0.086 0 0.0378" rpy="0 0 0" />
+      <mass value="0.4555" />
+      <inertia
+        ixx="0.00145" ixy="0" ixz="0.000124"
+        iyy="0.00233" iyz="0"
+        izz="0.00290" />
+    </inertial>
+    <visual>
+      <origin xyz="0 0 0" rpy="0 0 0" />
+      <geometry>
+        <mesh filename="${path_meshes}/body/base_link.STL" />
       </geometry>
       <material name="Yellow" />
@@ -90,10 +90,10 @@
   <link name="column_body_Link">
     <inertial>
-      <origin xyz="-0.10613 0.0015789 0.046254" rpy="0 0 0" />
-      <mass value="0.10507" />
-      <inertia
-        ixx="0.00033714" ixy="0" ixz="0"
-        iyy="0.00079716" iyz="0"
-        izz="0.0010369" />
+      <origin xyz="-0.11 0.00119 0.05782" rpy="0 0 0" />
+      <mass value="0.1397" />
+      <inertia
+        ixx="0.00048" ixy="0" ixz="0"
+        iyy="0.00098" iyz="0"
+        izz="0.00124" />
     </inertial>
     <visual>
@@ -182,5 +182,6 @@
   <!-- IMU -->
   <xacro:imu name="imu" parent="base_link">
-    <origin xyz="-0.06 0 0.11" rpy="0 0 0" />
+    <!--<origin xyz="-0.06 0 0.11" rpy="0 0 0" />-->
+    <origin xyz="-0.0617 -0.0008 0.1043376" rpy="0 0 0" />
   </xacro:imu>
   <!-- IMU -->

File: dude_description/urdf/imu.urdf.xacro (robot description, xacro)
@@ -3,8 +3,16 @@
   <xacro:macro name="imu" params="name parent *joint_pose">
     <link name="${name}_link">
+      <inertial>
+        <origin xyz="0.0002 0.003 -0.00025" rpy="0 0 0" />
+        <mass value="0.0045" />
+        <inertia
+          ixx="6.80127923442653E-07" ixy="2.58853590724977E-08" ixz="6.27330058259111E-09"
+          iyy="2.67621227004883E-07" iyz="3.00971478682596E-08"
+          izz="9.29933868272119E-07" />
+      </inertial>
       <visual>
         <origin xyz="0 0 0" rpy="0 0 0" />
         <geometry>
-          <box size="0.028 0.041 0.005" />
+          <mesh filename="${path_meshes}/imu/imu_Link.STL" />
         </geometry>
         <material name="Red" />
@@ -16,6 +24,4 @@
       <child link="${name}_link" />
     </joint>
-    <gazebo reference="${name}_link">
-    </gazebo>
-  </xacro:macro>
+ </xacro:macro>
 </robot>
