Commit message: Fixed initialization motors

File: dude_description/urdf/omniwheel.urdf.xacro (robot description, xacro)
@@ -39,5 +39,5 @@
       <child link="omniwheel_Link" />
       <axis xyz="0 -1 0" />
-      <mimic joint="Left" multiplier="1" offset="0"/>
+      <mimic joint="left_joint" multiplier="1" offset="0"/>
     </joint>
   </xacro:macro>
